File: 6_Test/2_PCB/test_board_dyl/analogsupply.kicad_sch (KiCad schematic)
At the start: 17 parts, among them U1 TPS74501PDRVR, U2 ADA4807-1AKSZ-R7, U3 ADA4807-1AKSZ-R7

Commit message: Clean up folder
Parts:
- L1: footprint IND_BLM18_0603_MUR -> ferriteBead120OhmFootprints:IND_BLM18_0603_MUR
- R10: value RC0402JR-071KL -> 6k
- R11, R14, R15: value 3310Y-001-103L -> 10k; footprint 3310Y-001-103L:TRIM_3310Y-001-103L -> potentiometer_10turn:potentiometer_10turn
- R13: value RC0402JR-071KL -> 1k
- U1: footprint DRV0006A -> tps745Footprints:DRV0006A_NV
- U2, U3: footprint KS-6_ADI -> opampADA4807Footprints:KS-6_ADI
Changed lines of the file:
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@@
 			)
 		)
-		(property "Value" "3310Y-001-103L"
+		(property "Value" "10k"
 			(at 165.1 104.1399 90)
 			(effects
@@
 			)
 		)
-		(property "Footprint" "3310Y-001-103L:TRIM_3310Y-001-103L"
+		(property "Footprint" "potentiometer_10turn:potentiometer_10turn"
 			(at 162.56 102.87 0)
 			(effects
@@
 			)
 		)
-		(property "Value" "RC0402JR-071KL"
+		(property "Value" "1k"
 			(at 160.02 78.7399 90)
 			(effects
@@
 			)
 		)
-		(property "Value" "3310Y-001-103L"
+		(property "Value" "10k"
 			(at 133.35 72.39 0)
 			(effects
@@
 			)
 		)
-		(property "Footprint" "3310Y-001-103L:TRIM_3310Y-001-103L"
+		(property "Footprint" "potentiometer_10turn:potentiometer_10turn"
 			(at 133.35 76.2 0)
 			(effects
@@
 			)
 		)
-		(property "Footprint" "DRV0006A"
+		(property "Footprint" "tps745Footprints:DRV0006A_NV"
 			(at 91.44 55.88 0)
 			(effects
@@
 			)
 		)
-		(property "Value" "RC0402JR-071KL"
+		(property "Value" "6k"
 			(at 128.27 60.9599 90)
 			(effects
@@
 			)
 		)
-		(property "Footprint" "KS-6_ADI"
+		(property "Footprint" "opampADA4807Footprints:KS-6_ADI"
 			(at 175.26 107.95 0)
 			(effects
@@
 			)
 		)
-		(property "Footprint" "KS-6_ADI"
+		(property "Footprint" "opampADA4807Footprints:KS-6_ADI"
 			(at 175.26 81.28 0)
 			(effects
@@
 			)
 		)
-		(property "Footprint" "IND_BLM18_0603_MUR"
+		(property "Footprint" "ferriteBead120OhmFootprints:IND_BLM18_0603_MUR"
 			(at 36.83 45.72 0)
 			(effects
@@
 			)
 		)
-		(property "Value" "3310Y-001-103L"
+		(property "Value" "10k"
 			(at 165.1 128.2699 90)
 			(effects
@@
 			)
 		)
-		(property "Footprint" "3310Y-001-103L:TRIM_3310Y-001-103L"
+		(property "Footprint" "potentiometer_10turn:potentiometer_10turn"
 			(at 162.56 127 0)
 			(effects
