File: 6_Test/2_PCB/test_board_dyl/digitalsupply.kicad_sch (KiCad schematic)
At the start: 10 parts, among them U5 TPS74501PDRVR

Commit message: Clean up folder
Parts:
- L2: footprint IND_BLM18_0603_MUR -> ferriteBead120OhmFootprints:IND_BLM18_0603_MUR
- R36, R38: footprint (none) -> Resistor_SMD:R_0201_0603Metric
- R37: footprint POT_PV37W_MUR -> potentiometer_10turn:potentiometer_10turn
- U5: footprint DRV0006A -> tps745Footprints:DRV0006A_NV
Changed lines of the file:
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@@
 			)
 		)
-		(property "Footprint" "IND_BLM18_0603_MUR"
+		(property "Footprint" "ferriteBead120OhmFootprints:IND_BLM18_0603_MUR"
 			(at 72.39 63.5 0)
 			(effects
@@
 			)
 		)
-		(property "Footprint" "POT_PV37W_MUR"
+		(property "Footprint" "potentiometer_10turn:potentiometer_10turn"
 			(at 176.53 95.25 0)
 			(effects
@@
 			)
 		)
-		(property "Footprint" "DRV0006A"
+		(property "Footprint" "tps745Footprints:DRV0006A_NV"
 			(at 142.24 73.66 0)
 			(effects
@@
 			)
 		)
-		(property "Footprint" ""
+		(property "Footprint" "Resistor_SMD:R_0201_0603Metric"
 			(at 177.546 99.314 90)
 			(effects
@@
 			)
 		)
-		(property "Footprint" ""
+		(property "Footprint" "Resistor_SMD:R_0201_0603Metric"
 			(at 177.546 71.374 90)
 			(effects
