File: 6_Test/2_PCB/test_board_1/schematics/board_main.kicad_sch (KiCad schematic)
At the start: 29 parts, among them J1 Digital_Outputs, J10 Analog_Inputs_Jumpers, J3 BNC1, J4 Digital_Inputs, J5 BNC_to_Analog, J6 BNC2, J7 Conn_02x06_Row_Letter_First, J8 IOVDD_Jumpers, J9 Power_Connector

Commit message: creating new project. combining work
Other:
- moved on the sheet: ADC_chip, ADC_socket, C10, C11, C12, C13, C14, C6, C7, C8, C9, J1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

Commit message: final draft of board done.
Parts:
- removed ADC_chip: ~, symbol chip:Chip
- removed ADC_socket: ~, Package_DIP:DIP-32_W15.24mm_Socket, symbol chip:Chip
- removed C10, C11, C6, C7, C8, C9: 100pF, symbol Device:C
- removed C12, C13: 4.7uF, symbol Device:C
- removed C14: 100nF, symbol Device:C
- removed J1: Digital_Outputs, symbol Connector_Generic:Conn_01x06
- removed J10: Analog_Inputs_Jumpers, symbol Connector_Generic:Conn_02x06_Row_Letter_First
- removed J3: BNC1, CONN_1274571-1_TYCO, symbol bnc_mini:1274571-1
- removed J4: Digital_Inputs, symbol Connector_Generic:Conn_01x08
- removed J5: BNC_to_Analog, symbol Connector_Generic:Conn_02x06_Row_Letter_First
- removed J6: BNC2, CONN_1274571-1_TYCO, symbol bnc_mini:1274571-1
- removed J7: Conn_02x06_Row_Letter_First, symbol Connector_Generic:Conn_02x06_Row_Letter_First
- removed J8: IOVDD_Jumpers, symbol Connector_Generic:Conn_02x04_Row_Letter_First
- removed J9: Power_Connector, symbol Connector_Generic:Conn_01x02
- removed R21, R22, R23, R24, R25, R26: 1k, symbol Device:R_US
- removed R27: 6k, symbol Device:R_US
- removed R28: 10k, POT_PV37W_MUR, symbol pot10turn:PV37W103C01B00
- removed R29: 4.7k, symbol Device:R_US
- added J? (x3): 67996-130HLF, 67996-130HLF_AMP, symbol 15x2Header:67996-130HLF
Other:
- added sheet ADC (ADC/ADC_final.kicad_sch)
- added sheet LDO_Cir (LDOCircuitry/LDO_circuitry_final.kicad_sch)
- added sheet ResetPulse (ResetPulse/reset_pulse_final.kicad_sch)
- sheet AnalogSupply: file analogsupply.kicad_sch -> AnalogSupply/analogSupply_final.kicad_sch
- sheet AnalogSupply ports: added VSUP; removed GND, V_SUP
- sheet Buffer: file buffer.kicad_sch -> Buffer/buffer_final.kicad_sch
- sheet Buffer ports: added CLKX, CLK_IND, CLK_OUT1, CLK_OUT2, CLK_OUT3, CLK_OUT4, CLK_OUT5, CLK_OUT6, RESX, RES_IND; removed CLK1, CLK2, CLK4, CLK5, CLK6, CLk3, RES, RES_IN
- sheet DigitalSupply: file digitalsupply.kicad_sch -> DigitalSupply/digitalSupply_final.kicad_sch
- sheet DigitalSupply ports: added VSUP; removed GND, V_SUP
- note added: "Analog Discovery"
- note added: "Digital Discovery1"
- note added: "Digital Discovery2"
