File: 6_Test/2_PCB/test_board_1/schematics/Buffer/buffer_final.kicad_sch (KiCad schematic)
At the start: 21 parts, among them U1 SN74ALVCH162827DLR

Commit message: final draft of board done.
Parts:
- removed R13, R14, R15, R16, R17, R18, R19, R20: 22, symbol Device:R_US
- added R? (x2): 22, Resistor_SMD:R_0402_1005Metric, symbol Device:R_US
- R1, R10, R11, R12, R2, R3, R4, R5, R6, R7, R8, R9: footprint (none) -> Resistor_SMD:R_0402_1005Metric
Connections:
- net DO15 is gone; now on net GND: U1.20 (2Y5)
- net DO16 is gone; now on net GND: U1.21 (2Y6)
- net DO17 is gone; now on net GND: U1.23 (2Y7)
- net DO18 is gone; now on net GND: U1.24 (2Y8)
- net DO19 is gone; now on net GND: U1.26 (2Y9)
- net DO20 is gone; now on net GND: U1.27 (2Y10)
- net GND: now also U1.30 (2A10), U1.31 (2A9), U1.33 (2A8), U1.34 (2A7), U1.36 (2A6), U1.37 (2A5)
- net at U1.38 (2A4): now also R?.2
- net at U1.40 (2A3): now also R?.2
- net DI10 renamed CLK_IN4
- net DI11 renamed CLK_IN5
- net DI12 renamed CLK_IN6
- net DI7 renamed CLK_IN1
- net DI8 renamed CLK_IN2
- net DI9 renamed CLK_IN3
- net DO10 renamed CLK_OUT4
- net DO11 renamed CLK_OUT5
- net DO12 renamed CLK_OUT6
- net DO13 renamed RESX
- net DO14 renamed CLKX
- net DO7 renamed CLK_OUT1
- net DO8 renamed CLK_OUT2
- net DO9 renamed CLK_OUT3
- new net CLK_IND: R?.1
- new net RES_IND: R?.1
