File: 6_Test/2_PCB/test_board_1/schematics/Buffer/digital_buffer_sim.kicad_sch (KiCad schematic)
At the start: 4 parts, among them U1 SN74ALVCH162827DLR

Commit message: final draft of board done.
Parts:
- removed V1: VPULSE, symbol Simulation_SPICE:VPULSE
- added V1: 2, symbol Simulation_SPICE:VDC
Connections:
- net GND: now also V1.2
- net vs: now also V1.1
