File: 6_Test/2_PCB/test_board_1/schematics/DigitalSupply/digitalSupply_final.kicad_sch (KiCad schematic)
At the start: 9 parts, among them U4 TPS74501PDRVR

Commit message: final draft of board done.
Parts:
- added R?: 4.7k, symbol Device:R
- R7: value 1k -> 4.7k; footprint Resistor_SMD:R_0402_1005Metric -> (none)
Connections:
- net GND: now also R?.2; no longer R8.1
- new net: R8.1, R?.1
Other:
- note removed: ".ac lin 100000 0 100000000"
Changed lines of the file:
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@@
+	(wire
+		(pts
+			(xy 198.12 120.65) (xy 198.12 125.73)
+		)
+		(stroke
+			(width 0)
+			(type default)
+		)
+	)
 	(wire
 		(pts
@@
 	(wire
 		(pts
-			(xy 198.12 109.22) (xy 198.12 118.11)
-		)
-		(stroke
-			(width 0)
-			(type default)
-		)
-	)
-	(wire
-		(pts
 			(xy 96.52 87.63) (xy 96.52 91.44)
 		)
@@
 	(wire
 		(pts
+			(xy 198.12 109.22) (xy 198.12 113.03)
+		)
+		(stroke
+			(width 0)
+			(type default)
+		)
+	)
+	(wire
+		(pts
 			(xy 198.12 87.63) (xy 198.12 88.9)
 		)
@@
 			(width 0)
 			(type default)
-		)
-	)
-	(text ".ac lin 100000 0 100000000"
-		(exclude_from_sim no)
-		(at 142.24 117.348 0)
-		(effects
-			(font
-				(size 1.27 1.27)
-			)
 		)
 	)
@@
 		(dnp no)
 		(fields_autoplaced yes)
-		(property "Reference" "#PWR09"
+		(property "Reference" "#PWR011"
 			(at 124.46 97.79 0)
 			(effects
@@
 			(project "digitalSupply_final"
 				(path "/9c0580c5-7bd5-4e54-bf4c-826aa4ac3630/67cdf4fb-e160-416a-a6f0-b53d0a3ad737"
-					(reference "#PWR09")
+					(reference "#PWR011")
 					(unit 1)
 				)
@@
 			)
 		)
-		(property "Value" "1k"
+		(property "Value" "4.7k"
 			(at 200.66 85.0899 0)
 			(effects
@@
 			)
 		)
-		(property "Footprint" "Resistor_SMD:R_0402_1005Metric"
+		(property "Footprint" ""
 			(at 196.342 83.82 90)
 			(effects
@@
 		(dnp no)
 		(fields_autoplaced yes)
-		(property "Reference" "#PWR010"
+		(property "Reference" "#PWR012"
 			(at 142.24 109.22 0)
 			(effects
@@
 			(project "digitalSupply_final"
 				(path "/9c0580c5-7bd5-4e54-bf4c-826aa4ac3630/67cdf4fb-e160-416a-a6f0-b53d0a3ad737"
-					(reference "#PWR010")
+					(reference "#PWR012")
 					(unit 1)
 				)
@@
 		(dnp no)
 		(fields_autoplaced yes)
-		(property "Reference" "#PWR08"
+		(property "Reference" "#PWR010"
 			(at 96.52 97.79 0)
 			(effects
@@
 			(project "digitalSupply_final"
 				(path "/9c0580c5-7bd5-4e54-bf4c-826aa4ac3630/67cdf4fb-e160-416a-a6f0-b53d0a3ad737"
-					(reference "#PWR08")
+					(reference "#PWR010")
 					(unit 1)
 				)
@@
 		(dnp no)
 		(fields_autoplaced yes)
-		(property "Reference" "#PWR011"
+		(property "Reference" "#PWR013"
 			(at 181.61 111.76 0)
 			(effects
@@
 			(project "digitalSupply_final"
 				(path "/9c0580c5-7bd5-4e54-bf4c-826aa4ac3630/67cdf4fb-e160-416a-a6f0-b53d0a3ad737"
-					(reference "#PWR011")
+					(reference "#PWR013")
 					(unit 1)
 				)
@@
 	(symbol
 		(lib_id "power:GND")
-		(at 198.12 118.11 0)
+		(at 198.12 125.73 0)
 		(unit 1)
 		(exclude_from_sim no)
@@
 		(dnp no)
 		(fields_autoplaced yes)
-		(property "Reference" "#PWR012"
-			(at 198.12 124.46 0)
+		(property "Reference" "#PWR014"
+			(at 198.12 132.08 0)
 			(effects
 				(font
@@
 		)
 		(property "Value" "GND"
-			(at 198.12 123.19 0)
+			(at 198.12 130.81 0)
 			(effects
 				(font
@@
 		)
 		(property "Footprint" ""
-			(at 198.12 118.11 0)
+			(at 198.12 125.73 0)
 			(effects
 				(font
@@
 		)
 		(property "Datasheet" ""
-			(at 198.12 118.11 0)
+			(at 198.12 125.73 0)
 			(effects
 				(font
@@
 		)
 		(property "Description" "Power symbol creates a global label with name \"GND\" , ground"
-			(at 198.12 118.11 0)
+			(at 198.12 125.73 0)
 			(effects
 				(font
@@
 			(project "digitalSupply_final"
 				(path "/9c0580c5-7bd5-4e54-bf4c-826aa4ac3630/67cdf4fb-e160-416a-a6f0-b53d0a3ad737"
-					(reference "#PWR012")
+					(reference "#PWR014")
 					(unit 1)
 				)
@@
 	)
 	(symbol
+		(lib_id "Device:R")
+		(at 198.12 116.84 0)
+		(unit 1)
+		(exclude_from_sim no)
+		(in_bom yes)
+		(on_board yes)
+		(dnp no)
+		(fields_autoplaced yes)
+		(property "Reference" "R?"
+			(at 200.66 115.5699 0)
+			(effects
+				(font
+					(size 1.27 1.27)
+				)
+				(justify left)
+			)
+		)
+		(property "Value" "4.7k"
+			(at 200.66 118.1099 0)
+			(effects
+				(font
+					(size 1.27 1.27)
+				)
+				(justify left)
+			)
+		)
+		(property "Footprint" ""
+			(at 196.342 116.84 90)
+			(effects
+				(font
+					(size 1.27 1.27)
+				)
+				(hide yes)
+			)
+		)
+		(property "Datasheet" "~"
+			(at 198.12 116.84 0)
+			(effects
+				(font
+					(size 1.27 1.27)
+				)
+				(hide yes)
+			)
+		)
+		(property "Description" "Resistor"
+			(at 198.12 116.84 0)
+			(effects
+				(font
+					(size 1.27 1.27)
+				)
+				(hide yes)
+			)
+		)
+		(pin "2"
+		)
+		(pin "1"
+		)
+		(instances
+			(project "board_main"
+				(path "/9c0580c5-7bd5-4e54-bf4c-826aa4ac3630/67cdf4fb-e160-416a-a6f0-b53d0a3ad737"
+					(reference "R?")
+					(unit 1)
+				)
+			)
+		)
+	)
+	(symbol
 		(lib_id "power:GND")
 		(at 220.98 86.36 0)
@@
 		(dnp no)
 		(fields_autoplaced yes)
-		(property "Reference" "#PWR013"
+		(property "Reference" "#PWR015"
 			(at 220.98 92.71 0)
 			(effects
@@
 			(project "digitalSupply_final"
 				(path "/9c0580c5-7bd5-4e54-bf4c-826aa4ac3630/67cdf4fb-e160-416a-a6f0-b53d0a3ad737"
-					(reference "#PWR013")
+					(reference "#PWR015")
 					(unit 1)
 				)
@@
 		(dnp no)
 		(fields_autoplaced yes)
-		(property "Reference" "#PWR014"
+		(property "Reference" "#PWR016"
 			(at 237.49 92.71 0)
 			(effects
@@
 			(project "digitalSupply_final"
 				(path "/9c0580c5-7bd5-4e54-bf4c-826aa4ac3630/67cdf4fb-e160-416a-a6f0-b53d0a3ad737"
-					(reference "#PWR014")
-					(unit 1)
-				)
+					(reference "#PWR016")
+					(unit 1)
+				)
