File: 6_Test/2_PCB/test_board_1/schematics/DigitalSupply/digitalSupply_final_sim.kicad_sch (KiCad schematic)
At the start: 10 parts, among them U1 TPS74501PDRVR

Commit message: final draft of board done.
Other:
- note removed: ".ac lin 100000 0 100000000"
Changed lines of the file:
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@@
-		)
-	)
-	(text ".ac lin 100000 0 100000000"
-		(exclude_from_sim no)
-		(at 142.24 117.348 0)
-		(effects
-			(font
-				(size 1.27 1.27)
-			)
 		)
 	)
