File: 6_Test/2_PCB/test_board_dyl/board_main/analogsupply.kicad_sch (KiCad schematic)
At the start: 16 parts, among them U2 ADA4807-2ARMZ, U5 TPS74501PDRVR

Commit message: creating new project. combining work
Parts:
- removed C15, C16, C17: 4.7u, Capacitor_SMD:C_0201_0603Metric, symbol Device:C
- removed C18, C20, C21: 100n, Capacitor_SMD:C_0201_0603Metric, symbol Device:C
- removed C19: C, Capacitor_SMD:C_0201_0603Metric, symbol Device:C
- removed L2: BLM18PG121SN1D, IND_BLM18_0603_MUR, symbol ferritebead:BLM18PG121SN1D
- removed R30, R33: R_US, symbol Device:R_US
- removed R31, R34, R35: 10k, POT_PV37W_MUR, symbol pot10turn:PV37W103C01B00
- removed R32: 8k, symbol Device:R_US
- removed U2: ADA4807-2ARMZ, RM-8_ADI, symbol opAmp:ADA4807-2ARMZ
- removed U5: TPS74501PDRVR, DRV0006A, symbol tps745:TPS74501PDRVR
- added C3, C? (x2): CL10A475KP8NNNC, CAP_0603_CL10A_1P6XP8_SAM, symbol Cap4.7uF:CL10A475KP8NNNC
- added C4, C5, C6, C7: CL05B104KP5NNNC, CAP_CL05_SAM, symbol Cap100nF:CL05B104KP5NNNC
- added L?: BLM18PG121SN1D, IND_BLM18_0603_MUR, symbol ferriteBeads120Ohm:BLM18PG121SN1D
- added R2, R5, R7: 3310Y-001-103L, 3310Y-001-103L:TRIM_3310Y-001-103L, symbol potentiometer:3310Y-001-103L
- added R3: ${SIM.PARAMS}, RC0402FR-074K7L:RESC1005X40, symbol resistor4.7k:RC0402FR-074K7L
- added R4, R?: RC0402JR-071KL, RC0402N_YAG, symbol Resistor1k:RC0402JR-071KL
- added U2, U3: ADA4807-1AKSZ-R7, KS-6_ADI, symbol Opamp:ADA4807-1AKSZ-R7
- added U?: TPS74501PDRVR, DRV0006A, symbol LDO:TPS74501PDRVR
Connections:
- net AVDD: now also C7.2, C?.1, R4.1, R?.1, U?.1 (OUT)
- net GND: now also C3.2, C5.1, C6.1, C7.1, C?.2, C?.2, R3.1, R5.2, U2.2 (-VS), U3.2 (-VS), U?.3 (GND)
- net VHI: now also C4.2, C5.2, U2.1 (VOUT), U2.4 (-IN)
- net VLO: now also C4.1, C6.2, U3.1 (VOUT), U3.4 (-IN)
- new net: R7.1, R?.2
- new net: R2.1, R4.2, U2.3 (+IN)
- new net: R2.2, R5.1, U3.3 (+IN)
- new net: R3.2, R7.2, U?.2 (FB)
- new net: C?.1, L?.1, U2.5 (*DISABLE), U2.6 (+VS), U3.5 (*DISABLE), U3.6 (+VS), U?.4 (EN), U?.6 (IN)
- new net Analog_Discover_Input: C3.1, L?.2

Commit message: progress on merging
Parts:
- renumbered U2 to U?
Connections:
- net GND: now also U?.7 (PAD); no longer C5.1, C6.1, R3.1, R5.2
- net Analog_Discover_Input renamed VSUP
- new net AVSS: C5.1, C6.1, R3.1, R5.2

Commit message: final draft of board done.
Parts:
- renumbered C4 to C?, C3 to C?, C5 to C?, C6 to C?, C7 to C?, R2 to R?, R7 to R?, R3 to R?, R4 to R?, R5 to R?, U3 to U?
Changed lines of the file:
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@@
 		(dnp no)
 		(fields_autoplaced yes)
-		(property "Reference" "#PWR022"
+		(property "Reference" "#PWR?"
 			(at 264.16 62.23 0)
 			(effects
@@
 		)
 		(instances
+			(project "board_main"
+				(path "/2f1c28d0-b53e-40e9-b5bc-17715b545373/c35211e2-8572-42d3-a6ba-25a7101b7bb6"
+					(reference "#PWR?")
+					(unit 1)
+				)
+			)
 			(project "test_board_1"
 				(path "/7acc191a-fe8c-48a0-9d8b-f697ef59ac03/c35211e2-8572-42d3-a6ba-25a7101b7bb6"
@@
 				)
 			)
+			(project "board_main"
+				(path "/2f1c28d0-b53e-40e9-b5bc-17715b545373/c35211e2-8572-42d3-a6ba-25a7101b7bb6"
+					(reference "R?")
+					(unit 1)
+				)
+			)
 			(project ""
 				(path "/bb4589bd-64fa-4400-9ba1-49fd7d1724b5"
@@
 		(dnp no)
 		(fields_autoplaced yes)
-		(property "Reference" "R2"
+		(property "Reference" "R?"
 			(at 177.8 99.0599 90)
 			(effects
@@
 		)
 		(instances
+			(project "board_main"
+				(path "/2f1c28d0-b53e-40e9-b5bc-17715b545373/c35211e2-8572-42d3-a6ba-25a7101b7bb6"
+					(reference "R?")
+					(unit 1)
+				)
+			)
 			(project "analogSupply_final_sim"
 				(path "/bb4589bd-64fa-4400-9ba1-49fd7d1724b5"
@@
 		(dnp no)
 		(fields_autoplaced yes)
-		(property "Reference" "R7"
+		(property "Reference" "R?"
 			(at 146.05 67.31 0)
 			(effects
@@
 		)
 		(instances
+			(project "board_main"
+				(path "/2f1c28d0-b53e-40e9-b5bc-17715b545373/c35211e2-8572-42d3-a6ba-25a7101b7bb6"
+					(reference "R?")
+					(unit 1)
+				)
+			)
 			(project ""
 				(path "/bb4589bd-64fa-4400-9ba1-49fd7d1724b5"
@@
 				)
 			)
+			(project "board_main"
+				(path "/2f1c28d0-b53e-40e9-b5bc-17715b545373/c35211e2-8572-42d3-a6ba-25a7101b7bb6"
+					(reference "C?")
+					(unit 1)
+				)
+			)
 			(project ""
 				(path "/bb4589bd-64fa-4400-9ba1-49fd7d1724b5"
@@
 		(dnp no)
 		(fields_autoplaced yes)
-		(property "Reference" "C4"
+		(property "Reference" "C?"
 			(at 252.73 97.7899 90)
 			(effects
@@
 		)
 		(instances
+			(project "board_main"
+				(path "/2f1c28d0-b53e-40e9-b5bc-17715b545373/c35211e2-8572-42d3-a6ba-25a7101b7bb6"
+					(reference "C?")
+					(unit 1)
+				)
+			)
 			(project "analogSupply_final_sim"
 				(path "/bb4589bd-64fa-4400-9ba1-49fd7d1724b5"
@@
 		(dnp no)
 		(fields_autoplaced yes)
-		(property "Reference" "C3"
+		(property "Reference" "C?"
 			(at 52.07 45.7199 90)
 			(effects
@@
 		)
 		(instances
+			(project "board_main"
+				(path "/2f1c28d0-b53e-40e9-b5bc-17715b545373/c35211e2-8572-42d3-a6ba-25a7101b7bb6"
+					(reference "C?")
+					(unit 1)
+				)
+			)
 			(project "analogSupply_final"
 				(path "/bb4589bd-64fa-4400-9ba1-49fd7d1724b5"
@@
 		(dnp no)
 		(fields_autoplaced yes)
-		(property "Reference" "R3"
+		(property "Reference" "R?"
 			(at 148.59 91.4399 90)
 			(effects
@@
 		)
 		(instances
+			(project "board_main"
+				(path "/2f1c28d0-b53e-40e9-b5bc-17715b545373/c35211e2-8572-42d3-a6ba-25a7101b7bb6"
+					(reference "R?")
+					(unit 1)
+				)
+			)
 			(project ""
 				(path "/bb4589bd-64fa-4400-9ba1-49fd7d1724b5"
@@
 		(dnp no)
 		(fields_autoplaced yes)
-		(property "Reference" "C5"
+		(property "Reference" "C?"
 			(at 264.16 86.3599 90)
 			(effects
@@
 		)
 		(instances
+			(project "board_main"
+				(path "/2f1c28d0-b53e-40e9-b5bc-17715b545373/c35211e2-8572-42d3-a6ba-25a7101b7bb6"
+					(reference "C?")
+					(unit 1)
+				)
+			)
 			(project "analogSupply_final_sim"
 				(path "/bb4589bd-64fa-4400-9ba1-49fd7d1724b5"
@@
 				)
 			)
+			(project "board_main"
+				(path "/2f1c28d0-b53e-40e9-b5bc-17715b545373/c35211e2-8572-42d3-a6ba-25a7101b7bb6"
+					(reference "#PWR?")
+					(unit 1)
+				)
+			)
 			(project ""
 				(path "/bb4589bd-64fa-4400-9ba1-49fd7d1724b5"
@@
 		(dnp no)
 		(fields_autoplaced yes)
-		(property "Reference" "U3"
+		(property "Reference" "U?"
 			(at 213.36 95.25 0)
 			(effects
@@
 		)
 		(instances
+			(project "board_main"
+				(path "/2f1c28d0-b53e-40e9-b5bc-17715b545373/c35211e2-8572-42d3-a6ba-25a7101b7bb6"
+					(reference "U?")
+					(unit 1)
+				)
+			)
 			(project ""
 				(path "/bb4589bd-64fa-4400-9ba1-49fd7d1724b5"
@@
 		(dnp no)
 		(fields_autoplaced yes)
-		(property "Reference" "R4"
+		(property "Reference" "R?"
 			(at 172.72 73.6599 90)
 			(effects
@@
 		)
 		(instances
+			(project "board_main"
+				(path "/2f1c28d0-b53e-40e9-b5bc-17715b545373/c35211e2-8572-42d3-a6ba-25a7101b7bb6"
+					(reference "R?")
+					(unit 1)
+				)
+			)
 			(project "analogSupply_final"
 				(path "/bb4589bd-64fa-4400-9ba1-49fd7d1724b5"
@@
 				)
 			)
+			(project "board_main"
+				(path "/2f1c28d0-b53e-40e9-b5bc-17715b545373/c35211e2-8572-42d3-a6ba-25a7101b7bb6"
+					(reference "U?")
+					(unit 1)
+				)
+			)
 			(project ""
 				(path "/bb4589bd-64fa-4400-9ba1-49fd7d1724b5"
@@
 		(dnp no)
 		(fields_autoplaced yes)
-		(property "Reference" "R5"
+		(property "Reference" "R?"
 			(at 177.8 123.1899 90)
 			(effects
@@
 		)
 		(instances
+			(project "board_main"
+				(path "/2f1c28d0-b53e-40e9-b5bc-17715b545373/c35211e2-8572-42d3-a6ba-25a7101b7bb6"
+					(reference "R?")
+					(unit 1)
+				)
+			)
 			(project "analogSupply_final_sim"
 				(path "/bb4589bd-64fa-4400-9ba1-49fd7d1724b5"
@@
 		(dnp no)
 		(fields_autoplaced yes)
-		(property "Reference" "#PWR0101"
+		(property "Reference" "#PWR?"
 			(at 77.47 62.23 0)
 			(effects
@@
 		)
 		(instances
+			(project "board_main"
+				(path "/2f1c28d0-b53e-40e9-b5bc-17715b545373/c35211e2-8572-42d3-a6ba-25a7101b7bb6"
+					(reference "#PWR?")
+					(unit 1)
+				)
+			)
 			(project "analogSupply_without_pots"
 				(path "/bb4589bd-64fa-4400-9ba1-49fd7d1724b5"
@@
 		)
 		(instances
+			(project "board_main"
+				(path "/2f1c28d0-b53e-40e9-b5bc-17715b545373/c35211e2-8572-42d3-a6ba-25a7101b7bb6"
+					(reference "U?")
+					(unit 1)
+				)
+			)
 			(project "opamp1_pot_low"
 				(path "/91b0f956-105d-46b2-b830-50f0dceaf9e9"
@@
 				)
 			)
+			(project "board_main"
+				(path "/2f1c28d0-b53e-40e9-b5bc-17715b545373/c35211e2-8572-42d3-a6ba-25a7101b7bb6"
+					(reference "C?")
+					(unit 1)
+				)
+			)
 			(project ""
 				(path "/bb4589bd-64fa-4400-9ba1-49fd7d1724b5"
@@
 		(dnp no)
 		(fields_autoplaced yes)
-		(property "Reference" "#PWR01"
+		(property "Reference" "#PWR?"
 			(at 48.26 64.77 0)
 			(effects
@@
 		)
 		(instances
+			(project "board_main"
+				(path "/2f1c28d0-b53e-40e9-b5bc-17715b545373/c35211e2-8572-42d3-a6ba-25a7101b7bb6"
+					(reference "#PWR?")
+					(unit 1)
+				)
+			)
 			(project "analogSupply_final"
 				(path "/bb4589bd-64fa-4400-9ba1-49fd7d1724b5"
@@
 		(dnp no)
 		(fields_autoplaced yes)
-		(property "Reference" "#PWR0107"
+		(property "Reference" "#PWR?"
 			(at 185.42 133.35 0)
 			(effects
@@
 		)
 		(instances
+			(project "board_main"
+				(path "/2f1c28d0-b53e-40e9-b5bc-17715b545373/c35211e2-8572-42d3-a6ba-25a7101b7bb6"
+					(reference "#PWR?")
+					(unit 1)
+				)
+			)
 			(project ""
 				(path "/bb4589bd-64fa-4400-9ba1-49fd7d1724b5"
@@
 		(dnp no)
 		(fields_autoplaced yes)
-		(property "Reference" "C6"
+		(property "Reference" "C?"
 			(at 264.16 113.0299 90)
 			(effects
@@
 		)
 		(instances
+			(project "board_main"
+				(path "/2f1c28d0-b53e-40e9-b5bc-17715b545373/c35211e2-8572-42d3-a6ba-25a7101b7bb6"
+					(reference "C?")
+					(unit 1)
+				)
+			)
 			(project "analogSupply_final"
 				(path "/bb4589bd-64fa-4400-9ba1-49fd7d1724b5"
@@
 		(dnp no)
 		(fields_autoplaced yes)
-		(property "Reference" "#PWR07"
+		(property "Reference" "#PWR?"
 			(at 233.68 62.23 0)
 			(effects
@@
 		)
 		(instances
+			(project "board_main"
+				(path "/2f1c28d0-b53e-40e9-b5bc-17715b545373/c35211e2-8572-42d3-a6ba-25a7101b7bb6"
+					(reference "#PWR?")
+					(unit 1)
+				)
+			)
 			(project "test_board_1"
 				(path "/7acc191a-fe8c-48a0-9d8b-f697ef59ac03/c35211e2-8572-42d3-a6ba-25a7101b7bb6"
@@
 				)
 			)
+			(project "board_main"
+				(path "/2f1c28d0-b53e-40e9-b5bc-17715b545373/c35211e2-8572-42d3-a6ba-25a7101b7bb6"
+					(reference "L?")
+					(unit 1)
+				)
+			)
 			(project ""
 				(path "/bb4589bd-64fa-4400-9ba1-49fd7d1724b5"
@@
 		(dnp no)
 		(fields_autoplaced yes)
-		(property "Reference" "C7"
+		(property "Reference" "C?"
 			(at 267.97 45.7199 90)
 			(effects
@@
 		)
 		(instances
+			(project "board_main"
+				(path "/2f1c28d0-b53e-40e9-b5bc-17715b545373/c35211e2-8572-42d3-a6ba-25a7101b7bb6"
+					(reference "C?")
+					(unit 1)
+				)
+			)
 			(project "analogSupply_final_sim"
 				(path "/bb4589bd-64fa-4400-9ba1-49fd7d1724b5"
