File: 6_Test/2_PCB/test_board_dyl/board_main/buffer.kicad_sch (KiCad schematic)
At the start: 21 parts, among them U1 SN74ALVCH162827DLR

Commit message: Fixed comments
Connections:
- net GND: now also R10.1, R11.1, R12.1, R13.1, R14.1, R7.1, R9.1, U1.10 (1Y7), U1.13 (1Y9), U1.14 (1Y10), U1.15 (2Y1), U1.16 (2Y2), U1.17 (2Y3), U1.19 (2Y4)
- net CLK_IN6: now reaches R20.1
- net CLK_IN5: now reaches R19.1
- net RES_IN: now reaches R8.1
- net CLK_IN3: now reaches R17.1
- net CLK_IN4: now reaches R18.1
- net CLK_IN2: now reaches R16.1
- net RES: now reaches U1.12 (1Y8)
- net CLK1: now reaches U1.20 (2Y5)
- net CLK2: now reaches U1.21 (2Y6)
- net CLk3: now reaches U1.23 (2Y7)
- net CLK4: now reaches U1.24 (2Y8)
- net CLK5: now reaches U1.26 (2Y9)
- net CLK6: now reaches U1.27 (2Y10)
- net CLK_IN1: now reaches R15.1

Commit message: final draft of board done.
Parts:
- renumbered R20 to R?, R11 to R?, R3 to R?, R19 to R?, R8 to R?, R6 to R?, R9 to R?, R17 to R?, R5 to R?, R4 to R?, R2 to R?, R12 to R?, R14 to R?, R1 to R?, R18 to R?, R13 to R?, R7 to R?, R16 to R?, R10 to R?, R15 to R?, U1 to U?
Changed lines of the file:
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@@
 		(on_board yes)
 		(dnp no)
-		(property "Reference" "R20"
+		(property "Reference" "R?"
 			(at 75.946 141.732 90)
 			(effects
@@
 		)
 		(instances
+			(project "board_main"
+				(path "/2f1c28d0-b53e-40e9-b5bc-17715b545373/8a0916ba-f0ff-4447-b0f5-57c87d76727c"
+					(reference "R?")
+					(unit 1)
+				)
+			)
 			(project "buffer"
 				(path "/e5075791-bb4a-4060-a781-4e8dd1df11ac"
@@
 		(on_board yes)
 		(dnp no)
-		(property "Reference" "R11"
+		(property "Reference" "R?"
 			(at 75.946 96.012 90)
 			(effects
@@
 		)
 		(instances
+			(project "board_main"
+				(path "/2f1c28d0-b53e-40e9-b5bc-17715b545373/8a0916ba-f0ff-4447-b0f5-57c87d76727c"
+					(reference "R?")
+					(unit 1)
+				)
+			)
 			(project "buffer"
 				(path "/e5075791-bb4a-4060-a781-4e8dd1df11ac"
@@
 		(on_board yes)
 		(dnp no)
-		(property "Reference" "R3"
+		(property "Reference" "R?"
 			(at 75.946 52.832 90)
 			(effects
@@
 		)
 		(instances
+			(project "board_main"
+				(path "/2f1c28d0-b53e-40e9-b5bc-17715b545373/8a0916ba-f0ff-4447-b0f5-57c87d76727c"
+					(reference "R?")
+					(unit 1)
+				)
+			)
 			(project "buffer"
 				(path "/e5075791-bb4a-4060-a781-4e8dd1df11ac"
@@
 		(on_board yes)
 		(dnp no)
-		(property "Reference" "R19"
+		(property "Reference" "R?"
 			(at 75.946 136.652 90)
 			(effects
@@
 		)
 		(instances
+			(project "board_main"
+				(path "/2f1c28d0-b53e-40e9-b5bc-17715b545373/8a0916ba-f0ff-4447-b0f5-57c87d76727c"
+					(reference "R?")
+					(unit 1)
+				)
+			)
 			(project "buffer"
 				(path "/e5075791-bb4a-4060-a781-4e8dd1df11ac"
@@
 		(on_board yes)
 		(dnp no)
-		(property "Reference" "R8"
+		(property "Reference" "R?"
 			(at 75.946 78.232 90)
 			(effects
@@
 		)
 		(instances
+			(project "board_main"
+				(path "/2f1c28d0-b53e-40e9-b5bc-17715b545373/8a0916ba-f0ff-4447-b0f5-57c87d76727c"
+					(reference "R?")
+					(unit 1)
+				)
+			)
 			(project "buffer"
 				(path "/e5075791-bb4a-4060-a781-4e8dd1df11ac"
@@
 		(on_board yes)
 		(dnp no)
-		(property "Reference" "R6"
+		(property "Reference" "R?"
 			(at 75.946 68.072 90)
 			(effects
@@
 		)
 		(instances
+			(project "board_main"
+				(path "/2f1c28d0-b53e-40e9-b5bc-17715b545373/8a0916ba-f0ff-4447-b0f5-57c87d76727c"
+					(reference "R?")
+					(unit 1)
+				)
+			)
 			(project "buffer"
 				(path "/e5075791-bb4a-4060-a781-4e8dd1df11ac"
@@
 		(on_board yes)
 		(dnp no)
-		(property "Reference" "R9"
+		(property "Reference" "R?"
 			(at 75.946 83.312 90)
 			(effects
@@
 		)
 		(instances
+			(project "board_main"
+				(path "/2f1c28d0-b53e-40e9-b5bc-17715b545373/8a0916ba-f0ff-4447-b0f5-57c87d76727c"
+					(reference "R?")
+					(unit 1)
+				)
+			)
 			(project "buffer"
 				(path "/e5075791-bb4a-4060-a781-4e8dd1df11ac"
@@
 		(on_board yes)
 		(dnp no)
-		(property "Reference" "R17"
+		(property "Reference" "R?"
 			(at 75.946 126.492 90)
 			(effects
@@
 		)
 		(instances
+			(project "board_main"
+				(path "/2f1c28d0-b53e-40e9-b5bc-17715b545373/8a0916ba-f0ff-4447-b0f5-57c87d76727c"
+					(reference "R?")
+					(unit 1)
+				)
+			)
 			(project "buffer"
 				(path "/e5075791-bb4a-4060-a781-4e8dd1df11ac"
@@
 		(on_board yes)
 		(dnp no)
-		(property "Reference" "R5"
+		(property "Reference" "R?"
 			(at 75.946 62.992 90)
 			(effects
@@
 		)
 		(instances
+			(project "board_main"
+				(path "/2f1c28d0-b53e-40e9-b5bc-17715b545373/8a0916ba-f0ff-4447-b0f5-57c87d76727c"
+					(reference "R?")
+					(unit 1)
+				)
+			)
 			(project "buffer"
 				(path "/e5075791-bb4a-4060-a781-4e8dd1df11ac"
@@
 		(on_board yes)
 		(dnp no)
-		(property "Reference" "R4"
+		(property "Reference" "R?"
 			(at 75.946 57.912 90)
 			(effects
@@
 		)
 		(instances
+			(project "board_main"
+				(path "/2f1c28d0-b53e-40e9-b5bc-17715b545373/8a0916ba-f0ff-4447-b0f5-57c87d76727c"
+					(reference "R?")
+					(unit 1)
+				)
+			)
 			(project "buffer"
 				(path "/e5075791-bb4a-4060-a781-4e8dd1df11ac"
@@
 		(on_board yes)
 		(dnp no)
-		(property "Reference" "R2"
+		(property "Reference" "R?"
 			(at 75.946 47.752 90)
 			(effects
@@
 		)
 		(instances
+			(project "board_main"
+				(path "/2f1c28d0-b53e-40e9-b5bc-17715b545373/8a0916ba-f0ff-4447-b0f5-57c87d76727c"
+					(reference "R?")
+					(unit 1)
+				)
+			)
 			(project "buffer"
 				(path "/e5075791-bb4a-4060-a781-4e8dd1df11ac"
@@
 		(on_board yes)
 		(dnp no)
-		(property "Reference" "R12"
+		(property "Reference" "R?"
 			(at 75.946 101.092 90)
 			(effects
@@
 		)
 		(instances
+			(project "board_main"
+				(path "/2f1c28d0-b53e-40e9-b5bc-17715b545373/8a0916ba-f0ff-4447-b0f5-57c87d76727c"
+					(reference "R?")
+					(unit 1)
+				)
+			)
 			(project "buffer"
 				(path "/e5075791-bb4a-4060-a781-4e8dd1df11ac"
@@
 		(on_board yes)
 		(dnp no)
-		(property "Reference" "R14"
+		(property "Reference" "R?"
 			(at 75.946 111.252 90)
 			(effects
@@
 		)
 		(instances
+			(project "board_main"
+				(path "/2f1c28d0-b53e-40e9-b5bc-17715b545373/8a0916ba-f0ff-4447-b0f5-57c87d76727c"
+					(reference "R?")
+					(unit 1)
+				)
+			)
 			(project "buffer"
 				(path "/e5075791-bb4a-4060-a781-4e8dd1df11ac"
@@
 		(on_board yes)
 		(dnp no)
-		(property "Reference" "R1"
+		(property "Reference" "R?"
 			(at 75.946 42.672 90)
 			(effects
@@
 		)
 		(instances
+			(project "board_main"
+				(path "/2f1c28d0-b53e-40e9-b5bc-17715b545373/8a0916ba-f0ff-4447-b0f5-57c87d76727c"
+					(reference "R?")
+					(unit 1)
+				)
+			)
 			(project ""
 				(path "/e5075791-bb4a-4060-a781-4e8dd1df11ac"
@@
 		(on_board yes)
 		(dnp no)
-		(property "Reference" "R18"
+		(property "Reference" "R?"
 			(at 75.946 131.572 90)
 			(effects
@@
 		)
 		(instances
+			(project "board_main"
+				(path "/2f1c28d0-b53e-40e9-b5bc-17715b545373/8a0916ba-f0ff-4447-b0f5-57c87d76727c"
+					(reference "R?")
+					(unit 1)
+				)
+			)
 			(project "buffer"
 				(path "/e5075791-bb4a-4060-a781-4e8dd1df11ac"
@@
 		(on_board yes)
 		(dnp no)
-		(property "Reference" "R13"
+		(property "Reference" "R?"
 			(at 75.946 106.172 90)
 			(effects
@@
 		)
 		(instances
+			(project "board_main"
+				(path "/2f1c28d0-b53e-40e9-b5bc-17715b545373/8a0916ba-f0ff-4447-b0f5-57c87d76727c"
+					(reference "R?")
+					(unit 1)
+				)
+			)
 			(project "buffer"
 				(path "/e5075791-bb4a-4060-a781-4e8dd1df11ac"
@@
 		(on_board yes)
 		(dnp no)
-		(property "Reference" "R7"
+		(property "Reference" "R?"
 			(at 75.946 73.152 90)
 			(effects
@@
 		)
 		(instances
+			(project "board_main"
+				(path "/2f1c28d0-b53e-40e9-b5bc-17715b545373/8a0916ba-f0ff-4447-b0f5-57c87d76727c"
+					(reference "R?")
+					(unit 1)
+				)
+			)
 			(project "buffer"
 				(path "/e5075791-bb4a-4060-a781-4e8dd1df11ac"
@@
 		(on_board yes)
 		(dnp no)
-		(property "Reference" "R16"
+		(property "Reference" "R?"
 			(at 75.946 121.412 90)
 			(effects
@@
 		)
 		(instances
+			(project "board_main"
+				(path "/2f1c28d0-b53e-40e9-b5bc-17715b545373/8a0916ba-f0ff-4447-b0f5-57c87d76727c"
+					(reference "R?")
+					(unit 1)
+				)
+			)
 			(project "buffer"
 				(path "/e5075791-bb4a-4060-a781-4e8dd1df11ac"
@@
 		(on_board yes)
 		(dnp no)
-		(property "Reference" "U1"
+		(property "Reference" "U?"
 			(at 152.4 49.53 0)
 			(effects
@@
 		)
 		(instances
+			(project "board_main"
+				(path "/2f1c28d0-b53e-40e9-b5bc-17715b545373/8a0916ba-f0ff-4447-b0f5-57c87d76727c"
+					(reference "U?")
+					(unit 1)
+				)
+			)
 			(project ""
 				(path "/e5075791-bb4a-4060-a781-4e8dd1df11ac"
@@
 		(on_board yes)
 		(dnp no)
-		(property "Reference" "R10"
+		(property "Reference" "R?"
 			(at 75.946 88.392 90)
 			(effects
@@
 		)
 		(instances
+			(project "board_main"
+				(path "/2f1c28d0-b53e-40e9-b5bc-17715b545373/8a0916ba-f0ff-4447-b0f5-57c87d76727c"
+					(reference "R?")
+					(unit 1)
+				)
+			)
 			(project "buffer"
 				(path "/e5075791-bb4a-4060-a781-4e8dd1df11ac"
@@
 		(on_board yes)
 		(dnp no)
-		(property "Reference" "R15"
+		(property "Reference" "R?"
 			(at 75.946 116.332 90)
 			(effects
@@
 		)
 		(instances
+			(project "board_main"
+				(path "/2f1c28d0-b53e-40e9-b5bc-17715b545373/8a0916ba-f0ff-4447-b0f5-57c87d76727c"
+					(reference "R?")
+					(unit 1)
+				)
+			)
 			(project "buffer"
 				(path "/e5075791-bb4a-4060-a781-4e8dd1df11ac"
