File: 6_Test/2_PCB/test_board_dyl/board_main/digitalsupply.kicad_sch (KiCad schematic)
At the start: 10 parts, among them U1 TPS74501PDRVR

Commit message: final draft of board done.
Parts:
- renumbered C3 to C?, C4 to C?, C1 to C?, C2 to C?, C5 to C?, L1 to L?, R1 to R?, R3 to R?, U1 to U?
Changed lines of the file:
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@@
 		(dnp no)
 		(fields_autoplaced yes)
-		(property "Reference" "C3"
+		(property "Reference" "C?"
 			(at 116.84 73.6599 0)
 			(effects
@@
 		)
 		(instances
+			(project "board_main"
+				(path "/2f1c28d0-b53e-40e9-b5bc-17715b545373/fdee9364-0143-49e5-8a4b-de9a4ad969eb"
+					(reference "C?")
+					(unit 1)
+				)
+			)
 			(project "digital_supply"
 				(path "/7eb40833-d3f4-415d-b3c4-00f1eb3abb07"
@@
 		(dnp no)
 		(fields_autoplaced yes)
-		(property "Reference" "C4"
+		(property "Reference" "C?"
 			(at 200.66 72.3899 0)
 			(effects
@@
 		)
 		(instances
+			(project "board_main"
+				(path "/2f1c28d0-b53e-40e9-b5bc-17715b545373/fdee9364-0143-49e5-8a4b-de9a4ad969eb"
+					(reference "C?")
+					(unit 1)
+				)
+			)
 			(project "digital_supply"
 				(path "/7eb40833-d3f4-415d-b3c4-00f1eb3abb07"
@@
 		(dnp no)
 		(fields_autoplaced yes)
-		(property "Reference" "R1"
+		(property "Reference" "R?"
 			(at 181.61 72.3899 0)
 			(effects
@@
 		)
 		(instances
+			(project "board_main"
+				(path "/2f1c28d0-b53e-40e9-b5bc-17715b545373/fdee9364-0143-49e5-8a4b-de9a4ad969eb"
+					(reference "R?")
+					(unit 1)
+				)
+			)
 			(project ""
 				(path "/7eb40833-d3f4-415d-b3c4-00f1eb3abb07"
@@
 		(dnp no)
 		(fields_autoplaced yes)
-		(property "Reference" "C1"
+		(property "Reference" "C?"
 			(at 72.39 73.6599 0)
 			(effects
@@
 		)
 		(instances
+			(project "board_main"
+				(path "/2f1c28d0-b53e-40e9-b5bc-17715b545373/fdee9364-0143-49e5-8a4b-de9a4ad969eb"
+					(reference "C?")
+					(unit 1)
+				)
+			)
 			(project ""
 				(path "/7eb40833-d3f4-415d-b3c4-00f1eb3abb07"
@@
 		(dnp no)
 		(fields_autoplaced yes)
-		(property "Reference" "R3"
+		(property "Reference" "R?"
 			(at 181.61 100.3299 0)
 			(effects
@@
 		)
 		(instances
+			(project "board_main"
+				(path "/2f1c28d0-b53e-40e9-b5bc-17715b545373/fdee9364-0143-49e5-8a4b-de9a4ad969eb"
+					(reference "R?")
+					(unit 1)
+				)
+			)
 			(project "digital_supply"
 				(path "/7eb40833-d3f4-415d-b3c4-00f1eb3abb07"
@@
 		(dnp no)
 		(fields_autoplaced yes)
-		(property "Reference" "C2"
+		(property "Reference" "C?"
 			(at 100.33 73.6599 0)
 			(effects
@@
 		)
 		(instances
+			(project "board_main"
+				(path "/2f1c28d0-b53e-40e9-b5bc-17715b545373/fdee9364-0143-49e5-8a4b-de9a4ad969eb"
+					(reference "C?")
+					(unit 1)
+				)
+			)
 			(project "digital_supply"
 				(path "/7eb40833-d3f4-415d-b3c4-00f1eb3abb07"
@@
 		(dnp no)
 		(fields_autoplaced yes)
-		(property "Reference" "L1"
+		(property "Reference" "L?"
 			(at 82.55 58.42 0)
 			(effects
@@
 		)
 		(instances
+			(project "board_main"
+				(path "/2f1c28d0-b53e-40e9-b5bc-17715b545373/fdee9364-0143-49e5-8a4b-de9a4ad969eb"
+					(reference "L?")
+					(unit 1)
+				)
+			)
 			(project ""
 				(path "/7eb40833-d3f4-415d-b3c4-00f1eb3abb07"
@@
 		(dnp no)
 		(fields_autoplaced yes)
-		(property "Reference" "C5"
+		(property "Reference" "C?"
 			(at 219.71 72.3899 0)
 			(effects
@@
 		)
 		(instances
+			(project "board_main"
+				(path "/2f1c28d0-b53e-40e9-b5bc-17715b545373/fdee9364-0143-49e5-8a4b-de9a4ad969eb"
+					(reference "C?")
+					(unit 1)
+				)
+			)
 			(project "digital_supply"
 				(path "/7eb40833-d3f4-415d-b3c4-00f1eb3abb07"
@@
 		(dnp no)
 		(fields_autoplaced yes)
-		(property "Reference" "U1"
+		(property "Reference" "U?"
 			(at 144.78 55.88 0)
 			(effects
@@
 		)
 		(instances
+			(project "board_main"
+				(path "/2f1c28d0-b53e-40e9-b5bc-17715b545373/fdee9364-0143-49e5-8a4b-de9a4ad969eb"
+					(reference "U?")
+					(unit 1)
+				)
+			)
 			(project ""
 				(path "/7eb40833-d3f4-415d-b3c4-00f1eb3abb07"
