File: 6_Test/2_PCB/test_board/schematics/DigitalSupply/digitalSupply_final.kicad_sch (KiCad schematic)
At the start: 10 parts, among them U4 TPS74501PDRVR

Commit message: Corrections to schematic 11_20_24
Parts:
- removed C10, C12: 100n, Capacitor_SMD:C_0402_1005Metric, symbol Device:C
- removed C11, C8, C9: 4.7u, Capacitor_SMD:C_0603_1608Metric, symbol Device:C
- removed L2: BLM18PG121SN1D, IND_BLM18_0603_MUR, symbol 2024-09-16_06-39-17:BLM18PG121SN1D
- removed R7, R?: 4.7k, symbol Device:R
- removed R8: PV37W103C01B00, PV37W103C01B00:TRIM_PV37W103C01B00, symbol pot_10turn:PV37W103C01B00
- removed U4: TPS74501PDRVR, DRV0006A, symbol TPS745_LDO:TPS74501PDRVR
- added C17, C18, C20: 4.7u, Capacitor_SMD:C_0201_0603Metric, symbol Device:C
- added C19, C21: 100n, Capacitor_SMD:C_0201_0603Metric, symbol Device:C
- added L2: BLM18PG121SN1D, ferriteBead120OhmFootprints:IND_BLM18_0603_MUR, symbol ferritebead:BLM18PG121SN1D
- added R16: 4.7k, Resistor_SMD:R_0201_0603Metric, symbol Device:R_US
- added R17: 10k, potentiometer_10turn:potentiometer_10turn, symbol pot10turn:PV37W103C01B00
- added R18: 6k, Resistor_SMD:R_0201_0603Metric, symbol Device:R_US
- added U4: LDO_Digital_Supply, tps745Footprints:DRV0006A_NV, symbol tps745:TPS74501PDRVR
Connections:
- net GND: now also C17.2, C18.2, C19.2, C20.2, C21.2, R18.2, U4.3 (GND), U4.5 (PG), U4.7 (PAD)
- net IOVDD: now also C18.1, C19.1, L2.1, U4.4 (EN), U4.6 (IN)
- net VDD: now also C20.1, C21.1, R16.1, U4.1 (OUT)
- new net: R16.2, R17.3
- new net: R17.1, R18.1
- new net: R17.2, U4.2 (FB)
- new net V_SUP: C17.1, L2.2
