File: 6_Test/2_PCB/test_board/schematics/DigitalSupply/digitalSupply_final.kicad_sch (KiCad schematic)
At the start: 8 parts, among them U4 TPS74501PDRVR

Commit message: final draft of board, revision 2
Parts:
- C10: footprint cap100nFFootprints:CAP_CL05_SAM -> Capacitor_SMD:C_0402_1005Metric
- R7, R9: footprint ECE628_lib:resistor4.7k -> Resistor_SMD:R_0402_1005Metric
Changed lines of the file:
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@@
 			)
 		)
-		(property "Footprint" "cap100nFFootprints:CAP_CL05_SAM"
+		(property "Footprint" "Capacitor_SMD:C_0402_1005Metric"
 			(at 121.6152 82.55 0)
 			(effects
@@
 			)
 		)
-		(property "Footprint" "ECE628_lib:resistor4.7k"
+		(property "Footprint" "Resistor_SMD:R_0402_1005Metric"
 			(at 185.674 78.994 90)
 			(effects
@@
 			)
 		)
-		(property "Footprint" "ECE628_lib:resistor4.7k"
+		(property "Footprint" "Resistor_SMD:R_0402_1005Metric"
 			(at 195.834 101.854 90)
 			(effects

Commit message: DRC passing with all our components and pcbway rules
Parts:
- U4: footprint tps745Footprints:DRV0006A -> tps745Footprints:DRV0006A_NV
Changed lines of the file:
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@@
 			)
 		)
-		(property "Footprint" "tps745Footprints:DRV0006A"
+		(property "Footprint" "tps745Footprints:DRV0006A_NV"
 			(at 152.4 81.28 0)
 			(effects
