File: 6_Test/2_PCB/test_board/schematics/AnalogSupply/analogSupply_final.kicad_sch (KiCad schematic)
At the start: 17 parts

Commit message: Edits 112524
Parts:
- C? (x4): value CL05B104KP5NNNC -> 100n; footprint CAP_CL05_SAM -> cap100nFFootprints:CAP_CL05_SAM
- C? (x3): value CL10A475KP8NNNC -> 4.7u; footprint CAP_0603_CL10A_1P6XP8_SAM -> Cap4.7uFFootprints:CAP_0603_CL10A_1P6XP8_SAM
- L?: footprint IND_BLM18_0603_MUR -> ferriteBead120OhmFootprints:IND_BLM18_0603_MUR
- R? (x2): value RC0402JR-071KL -> 1k
- R? (x3): value PV37W103C01B00 -> 10k; footprint PV37W103C01B00:TRIM_PV37W103C01B00 -> ECE628_lib:potentiometer_10turn
- U? (x2): footprint KS-6_ADI -> opampADA4807Footprints:KS-6_ADI
- U?: footprint DRV0006A -> tps745Footprints:DRV0006A
Other:
- moved on the sheet: C?, R?
