File: 6_Test/2_PCB/test_board/schematics/AnalogSupply/analogSupply_final.kicad_sch (KiCad schematic)
At the start: 17 parts

Commit message: final draft of board, revision 2
Parts:
- C? (x4): footprint cap100nFFootprints:CAP_CL05_SAM -> Capacitor_SMD:C_0402_1005Metric
- C? (x3): footprint Cap4.7uFFootprints:CAP_0603_CL10A_1P6XP8_SAM -> Capacitor_SMD:C_0603_1608Metric
- R? (x2): footprint RC0402N_YAG -> Resistor_SMD:R_0402_1005Metric
- R?: footprint RC0402FR-074K7L:RESC1005X40 -> Resistor_SMD:R_0402_1005Metric
Changed lines of the file:
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@@
 			)
 		)
-		(property "Footprint" "RC0402N_YAG"
+		(property "Footprint" "Resistor_SMD:R_0402_1005Metric"
 			(at 158.75 82.55 0)
 			(effects
@@
 			)
 		)
-		(property "Footprint" "RC0402N_YAG"
+		(property "Footprint" "Resistor_SMD:R_0402_1005Metric"
 			(at 127 64.77 0)
 			(effects
@@
 			)
 		)
-		(property "Footprint" "RC0402FR-074K7L:RESC1005X40"
+		(property "Footprint" "Resistor_SMD:R_0402_1005Metric"
 			(at 137.16 93.98 0)
 			(effects
@@
 			)
 		)
-		(property "Footprint" "cap100nFFootprints:CAP_CL05_SAM"
+		(property "Footprint" "Capacitor_SMD:C_0402_1005Metric"
 			(at 248.92 92.71 0)
 			(effects
@@
 			)
 		)
-		(property "Footprint" "cap100nFFootprints:CAP_CL05_SAM"
+		(property "Footprint" "Capacitor_SMD:C_0402_1005Metric"
 			(at 252.73 52.07 0)
 			(effects
@@
 			)
 		)
-		(property "Footprint" "cap100nFFootprints:CAP_CL05_SAM"
+		(property "Footprint" "Capacitor_SMD:C_0402_1005Metric"
 			(at 237.49 104.14 0)
 			(effects
@@
 			)
 		)
-		(property "Footprint" "cap100nFFootprints:CAP_CL05_SAM"
+		(property "Footprint" "Capacitor_SMD:C_0402_1005Metric"
 			(at 248.92 124.46 0)
 			(effects
@@
 			)
 		)
-		(property "Footprint" "Cap4.7uFFootprints:CAP_0603_CL10A_1P6XP8_SAM"
+		(property "Footprint" "Capacitor_SMD:C_0603_1608Metric"
 			(at 66.04 44.45 0)
 			(effects
@@
 			)
 		)
-		(property "Footprint" "Cap4.7uFFootprints:CAP_0603_CL10A_1P6XP8_SAM"
+		(property "Footprint" "Capacitor_SMD:C_0603_1608Metric"
 			(at 222.25 44.45 0)
 			(effects
@@
 			)
 		)
-		(property "Footprint" "Cap4.7uFFootprints:CAP_0603_CL10A_1P6XP8_SAM"
+		(property "Footprint" "Capacitor_SMD:C_0603_1608Metric"
 			(at 36.83 44.45 0)
 			(effects

Commit message: DRC passing with all our components and pcbway rules
Parts:
- U?: footprint tps745Footprints:DRV0006A -> tps745Footprints:DRV0006A_NV
Changed lines of the file:
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@@
 			)
 		)
-		(property "Footprint" "tps745Footprints:DRV0006A"
+		(property "Footprint" "tps745Footprints:DRV0006A_NV"
 			(at 92.71 54.61 0)
 			(effects

Commit message: Edit Layout 1_27
Rearranged the components in the layout and added majority of traces and ground layer. AVSS connections still need to be connected along with IOVDD
Parts:
- R?: value ${SIM.PARAMS} -> r=4.7k
Changed lines of the file:
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@@
 			)
 		)
-		(property "Value" "${SIM.PARAMS}"
+		(property "Value" "r=4.7k"
 			(at 139.7 95.2499 90)
 			(effects
