File: 6_Test/2_PCB/test_board/schematics/LDOCircuitry/LDO_circuitry_final.kicad_sch (KiCad schematic)
At the start: 6 parts

Commit message: Finished board layout
Parts:
- renumbered C35 to C31, C37 to C32, C36 to C33
Changed lines of the file:
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@@
 		(dnp no)
 		(fields_autoplaced yes)
-		(property "Reference" "C37"
+		(property "Reference" "C32"
 			(at 153.67 109.2199 0)
 			(effects
@@
 			(project "board_main"
 				(path "/9c0580c5-7bd5-4e54-bf4c-826aa4ac3630/104c40d7-ae25-447b-8675-a765b7f78bca"
-					(reference "C37")
+					(reference "C32")
 					(unit 1)
 				)
@@
 		(on_board yes)
 		(dnp no)
-		(property "Reference" "C35"
+		(property "Reference" "C31"
 			(at 125.984 102.616 0)
 			(effects
@@
 			(project "board_main"
 				(path "/9c0580c5-7bd5-4e54-bf4c-826aa4ac3630/104c40d7-ae25-447b-8675-a765b7f78bca"
-					(reference "C35")
+					(reference "C31")
 					(unit 1)
 				)
@@
 		(on_board yes)
 		(dnp no)
-		(property "Reference" "C36"
+		(property "Reference" "C33"
 			(at 141.224 108.966 0)
 			(effects
@@
 			(project "board_main"
 				(path "/9c0580c5-7bd5-4e54-bf4c-826aa4ac3630/104c40d7-ae25-447b-8675-a765b7f78bca"
-					(reference "C36")
-					(unit 1)
-				)
+					(reference "C33")
+					(unit 1)
+				)
